File: HW/pulseoximeter.kicad_sch (KiCad schematic)
At the start: 45 parts, among them J1 X05A20L15T, J2 TYPE-C-31-M-12, U1 TPD2EUSB30DRTR, U2 TPS7A4700RGWR, U3 ESP32-S3-MINI-1-N8, U4 LM324, U6 OPA140AIDBVR

Commit message: implemented dynamic chart y-axis scaling
Parts:
- removed C13, C7: 0.1uF, Capacitor_SMD:C_0402_1005Metric, symbol Device:C
- removed C18: 440pF, Capacitor_SMD:C_0603_1608Metric, symbol Device:C
- removed C8: 1uF, Capacitor_Tantalum_SMD:CP_EIA-3216-10_Kemet-I, symbol Device:C
- removed D1: D_Photo, LED_THT:LED_D3.0mm, symbol Device:D_Photo
- removed D2, D3, D6: LED, LED_THT:LED_D3.0mm, symbol Device:LED
- removed MOSFET1: DMN2310UT-13, Package_TO_SOT_SMD:SOT-523, symbol 2N7002:2N7002
- removed R11: 8.1M, Resistor_SMD:R_0603_1608Metric, symbol Device:R
- removed R15, R17: 10k, Resistor_SMD:R_0402_1005Metric, symbol Device:R
- removed R2: 1M, Resistor_SMD:R_0402_1005Metric, symbol Device:R
- removed R22: 330, Resistor_SMD:R_0603_1608Metric, symbol Device:R
- added C9: 0.1uF, Capacitor_SMD:C_0603_1608Metric, symbol Device:C
- added D2: D_Photo, LED_THT:LED_D3.0mm, symbol Device:D_Photo
- added J3, J4: Conn_01x02, Connector_PinHeader_2.54mm:PinHeader_1x02_P2.54mm_Vertical, symbol Connector_Generic:Conn_01x02
- added J5: Conn_01x01_Socket, Connector_PinHeader_2.54mm:PinHeader_1x01_P2.54mm_Vertical, symbol Connector:Conn_01x01_Socket
- added JP1, JP2, JP3, JP4: SolderJumper_2_Open, Jumper:SolderJumper-2_P1.3mm_Open_RoundedPad1.0x1.5mm, symbol Jumper:SolderJumper_2_Open
- added TP1, TP2, TP3: TestPoint, TestPoint:TestPoint_Pad_D2.0mm, symbol Connector:TestPoint
- added U5: TLC59116IPWR, PW28, symbol TLC59116IPWR:TLC59116IPWR
- added U7: LMC6001BIN/NOPB, LMC6001BIN_NOPB:DIP794W45P254L959H508Q8, symbol LMC6001BIN_NOPB:LMC6001BIN_NOPB
- C1, C2, C3: footprint Capacitor_SMD:C_0402_1005Metric -> Capacitor_SMD:C_0603_1608Metric
- C6: value 10uF -> 0.22uF; footprint Capacitor_SMD:C_0402_1005Metric -> Capacitor_SMD:C_0603_1608Metric
- D4: footprint LED_SMD:LED_0603_1608Metric -> LED_THT:LED_D3.0mm
- R1: value 10k -> 0; footprint Resistor_SMD:R_0402_1005Metric -> Resistor_SMD:R_0603_1608Metric
- R10, R4, R6, R9: footprint Resistor_SMD:R_0402_1005Metric -> Resistor_SMD:R_0603_1608Metric
- R12: value 33k -> 22k; footprint Resistor_SMD:R_0603_1608Metric -> Resistor_SMD:R_0805_2012Metric
- R13: value 330 -> 10k
- R14: value 330 -> 5.6M; footprint Resistor_SMD:R_0603_1608Metric -> Resistor_SMD:R_0805_2012Metric
- R3: value 1k -> 10k
- R7: value 330 -> 910
- U6: footprint OPA140AIDBVR:DBV5-M -> DBV5
Connections:
- net LEDK is gone; now on net SDA: J1.2
- net +3.3V: now also J1.12, J1.13, J1.6, R13.2, R3.1, JP1.1 (A), JP4.1 (A), TP3.1, U5.28 (VCC), U7.7 (V+); no longer J1.10, J1.3, J1.4
- net DISPLAY_CLK: now also J1.9, U3.18 (IO14); no longer J1.7, U3.16 (IO12)
- net DISPLAY_CS: now also J1.10, U3.17 (IO13); no longer J1.6, U3.14 (IO10)
- net DISPLAY_D/C: now also J1.11, U3.16 (IO12); no longer J1.5, U3.17 (IO13)
- net DISPLAY_RESET: now also J1.7, U3.20 (IO16); no longer J1.9, U3.18 (IO14)
- net DISPLAY_SDI: now also U3.19 (IO15); no longer U3.15 (IO11)
- net DN: no longer U1.1 (D+)
- net DP: now also U1.1 (D+)
- net GND: now also J1.15, J1.5, R1.1, R7.1, C9.2, D2.1 (K), J3.2 (Pin_2), U5.10 (GND), U5.19 (GND), U5.2 (A0), U5.24 (GND), U5.3 (A1), U5.4 (A2), U5.5 (A3), U7.4 (V-); no longer C6.2, D4.1 (K), D5.1 (K), J1.1, J1.11
- net HR_SIGNAL: now also JP2.1 (A)
- net SCL: now also J1.1, U5.26 (SCL); no longer J1.15
- net SDA: now also U5.27 (SDA); no longer J1.14
- net TP_INT: now also J1.3, U3.22 (IO18); no longer J1.13, U3.20 (IO16)
- net TP_RST: now also J1.4, U3.21 (IO17); no longer J1.12, U3.19 (IO15)
- net VBUS: now also D4.2 (A), D5.2 (A); no longer C6.1, R13.1, R14.1, R3.1, R7.1, U4.4 (V+), U6.5 (V+)
- net VCC/2: now also U4.13 (-), U4.3 (+), JP3.1 (A), U7.3 (IN+); no longer U4.12 (+), U4.2 (-), U6.3 (IN+)
- net at C20.2, R23.1, R24.2: now also U4.2 (-); no longer U4.3 (+)
- net IO0: now reaches U3.4 (IO0)
- net IO0: now also J3.1 (Pin_1)
- net at R7.2: now also U5.1 (REXT); no longer D5.2 (A)
- net at R12.2: now also R14.1, U7.6 (OUT); no longer U6.1 (OUT)
- net VDD_SPI_V: now reaches U3.41 (IO45)
- net VDD_SPI_V: now also J4.2 (Pin_2)
- net ROM_MSG: now reaches U3.44 (IO46)
- net ROM_MSG: now also J4.1 (Pin_1)
- net at U3.45 (EN): now also R3.2, C9.1
- net at R10.1, R9.2: now also U4.12 (+); no longer U4.13 (-)
- net at U6.4 (IN-): now also TP2.1
- net at R14.2: now also C6.2, U7.2 (IN-)
- net BACKLIGHT_EN: no longer names the net of U3.27 (IO47)
- net BACKLIGHT_EN: no longer R1.2
- net ESP32_RX: no longer names the net of U3.39 (TXD0)
- net ESP32_TX: no longer names the net of U3.40 (RXD0)
- new net: JP3.2 (B), U6.3 (IN+)
- new net: D5.1 (K), U5.9 (*OUT3)
- new net: J1.14, R1.2
- new net: JP1.2 (B), U4.4 (V+)
- new net: JP4.2 (B), U6.5 (V+)
- new net: J5.1 (Pin_1), JP2.2 (B)
- new net: C6.1, D2.2 (A)
- new net: TP1.1, U6.1 (OUT)
- new net: D4.1 (K), U5.14 (*OUT7)
- new net LED_RST: R13.1, U3.15 (IO11), U5.25 (*RESET)
- no-connect marks 35 -> 49
Other:
- moved on the sheet: C20, J2, R10, R23, R24, R5, R8, R9, U1, U4A, U4D, U4E
